File: PSFB_MCU.kicad_sch (KiCad schematic)
At the start: 135 parts, among them J2 Power_IN, Q1 WMM043N10HGD, Q2 WMM043N10HGD, Q3 WMM043N10HGD, Q4 WMM043N10HGD, U17 TLV3501AIDBV, U18 74LVC1G332, U19 TLV3501AIDBV, U20 TLV3501AIDBV, U4 AMS1117-5.0, U5 AMS1117-3.3, U6 LM5176PWP, Y1 16M

Commit message: VER1.0: добавил защиту бортового питания для тестов по ISO 7637-2 (Степень III)
Parts:
- removed U18: 74LVC1G332, symbol 74xGxx:74LVC1G332
- added C104: 10n, Capacitor_SMD:C_0805_2012Metric_Pad1.18x1.45mm_HandSolder, symbol Device:C_Small
- added D26: TD301MCANFD, MORNSUN:TD5(3)01MCANFD, symbol MORNSUN:TD5(3)01MCANFD
- added D41, D42: (no value), Package_TO_SOT_SMD:SOT-23, symbol Device:D_Dual_Series_AKC_Parallel
- added D45: (no value), Package_TO_SOT_SMD:SOT-23, symbol Power_Protection:NUP2105L
- added D46: D_TVS_Small, Diode_SMD:D_SMB, symbol Device:D_TVS_Small
- added D47: D_Small, Diode_SMD:D_SMB, symbol Device:D_Small
- added L14: (no value), Inductor_SMD:L_CommonModeChoke_TDK_ACM2520-2P, symbol Device:L_Coupled_Small
- added R98: 59, Resistor_SMD:R_0805_2012Metric_Pad1.20x1.40mm_HandSolder, symbol Device:R_Small
- C96: value 100n -> 10u; footprint Capacitor_SMD:C_0805_2012Metric_Pad1.18x1.45mm_HandSolder -> Capacitor_SMD:C_1206_3216Metric_Pad1.33x1.80mm_HandSolder
- C97: value 10p -> 100n; footprint Capacitor_SMD:C_0805_2012Metric_Pad1.18x1.45mm_HandSolder -> Capacitor_SMD:C_1206_3216Metric_Pad1.33x1.80mm_HandSolder
- D12: footprint Diode_SMD:D_SMB_Handsoldering -> Diode_SMD:D_SMC
- R78: value 0 -> 10; footprint Resistor_SMD:R_0805_2012Metric_Pad1.20x1.40mm_HandSolder -> Resistor_SMD:R_1206_3216Metric_Pad1.30x1.75mm_HandSolder; now fitted
- R86: value 100 -> 59
Connections:
- net CAN_RXD_MCU is gone; now on net CAN1_RXD_MCU: U3.44 (PA11)
- net CAN_TXD_MCU is gone; now on net CAN1_TXD_MCU: U3.45 (PA12)
- net DAC3 is gone; now on net DAC2: R89.1
- net ERROR_LvL1 is gone; now on net DAC2: U3.21 (PA5)
- net ERROR_LvL3 is gone; now on net TMR8_CH1N: U3.23 (PA7)
- net GPIO2 is gone; now on net TMR1_CH1N: U3.34 (PB13)
- net GPIO3 is gone; now on net TMR8_CH2N: U3.35 (PB14)
- net GPIO5 is gone; now on net TMR8_CH1: U3.37 (PC6)
- net GPIO6 is gone; now on net TMR8_CH2: U3.38 (PC7)
- net OverCurrent_1 is gone; now on net BkIN_1: C90.1, R81.1
- net OverCurrent_2 is gone; now on net BkIN_8: C98.1, R87.1
- net RS_TXD_MCU is gone; now on net TMR1_CH2: U3.42 (PA9)
- net Solenoid1_MCU is gone; now on net EEPROM_~{CS_MCU}: U3.50 (PA15)
- net Solenoid2_MCU is gone; now on net EEPROM_SCK_MCU: U3.51 (PC10)
- net Solenoid3_MCU is gone; now on net EEPROM_MISO_MCU: U3.52 (PC11)
- net Solenoid4_MCU is gone; now on net EEPROM_MOSI_MCU: U3.53 (PC12)
- net +3.3V: now also C96.1, C97.1, D26.4 (VCC), D41.2 (K), D42.2 (K); no longer C96.2
- net Current_measure_1: now also U3.16 (PA2)
- net Current_measure_2: now also U3.17 (PA3)
- net DAC1: now also R83.1, U3.20 (PA4); no longer R78.1
- net DAC2: no longer R83.1
- net GND: now also C96.2, D26.3 (GND), D41.1 (A), D42.1 (A); no longer C96.1
- net GND_IN: now also D46.1 (A1)
- net HVDC_MCU: now also U3.14 (PA0)
- net LVDC_MCU: now also U3.15 (PA1)
- net OverVoltage: now also D40.3 (common)
- net SHDN_OverCurrent_1: now also U3.9 (PC1)
- net SHDN_OverCurrent_2: now also U3.10 (PC2)
- net SHDN_OverVoltage: now also U3.8 (PC0)
- net TMR1_CH1: now also U3.41 (PA8)
- net TMR1_CH2N: now also U3.26 (PB0)
- net VIN: now also D47.2 (A); no longer L2.1
- net VIN_filtered: now also R78.2, D46.2 (A2); no longer C21.2, C22.1, C23.2, D12.2 (A2), L2.2, Q1.2 (D)
- net at C88.1, R52.1, R64.2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: no longer R78.2
- net CAN2_RXD_MCU: now reaches U3.57 (PB5)
- net CAN2_RXD_MCU: now also D26.1 (RXD)
- net CAN2_TXD_MCU: now reaches U3.58 (PB6)
- net CAN2_TXD_MCU: now also D26.2 (TXD)
- net at R86.2: now also D26.7 (CANH), L14.1
- removed net BkIN: C97.1, D40.3 (common), R86.1
- net CANH renamed CANH_1
- net CANL renamed CANL_1
- net ERROR_LvL2 renamed BkIN_1
- net BkIN_1: now also D41.3 (common)
- net GND_CAN renamed GND_CAN1
- net GPIO1 renamed BkIN_8
- net BkIN_8: now also D42.3 (common)
- net GPIO4: no longer names the net of U3.36 (PB15)
- net GPIO7: no longer names the net of U3.39 (PC8)
- net GPIO8: no longer names the net of U3.40 (PC9)
- net RS_RXD_MCU: no longer names the net of U3.43 (PA10)
- new net: C104.1, R86.1, R98.2
- new net: C21.2, C22.1, C23.2, D12.2 (A2), L2.2, Q1.2 (D), R78.1
- new net: D26.6 (CANL), L14.3, R98.1
- new net: D47.1 (K), L2.1
- new net CANH_2: D45.1 (K), L14.2
- new net CANL_2: D45.2 (K), L14.4
- new net GND_CAN2: C104.2, D26.5 (CANG), D45.3 (A)
- no-connect marks 10 -> 5
Other:
- note added: "CAN 1"
- note added: "CAN 2"
- note removed: "CAN"
- moved on the sheet: C100, C101, C88, C89, C90, C91, C92, C93, C94, C95, C98, C99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
