File: PSFB_MCU.kicad_sch (KiCad schematic)
At the start: 143 parts, among them J2 Power_IN, Q1 WMM043N10HGD, Q2 WMM043N10HGD, Q3 WMM043N10HGD, Q4 WMM043N10HGD, U17 TLV3501AIDBV, U19 TLV3501AIDBV, U20 TLV3501AIDBV, U4 AMS1117-5.0, U5 AMS1117-3.3, U6 LM5176PWP, Y1 16M

Commit message: VER1.0: добавил разделение питания VDD и VDDA
Parts:
- added C10, C9: 10u, Capacitor_SMD:C_0805_2012Metric_Pad1.18x1.45mm_HandSolder, symbol Device:C_Small
- added FB1: (no value), Inductor_SMD:L_0805_2012Metric_Pad1.05x1.20mm_HandSolder, symbol Device:FerriteBead_Small
- C1: renamed from C5; Description P/N (none) -> Capacitor SMD 25V
- C11: renamed from C1; Description P/N (none) -> Capacitor SMD 25V
- C12: renamed from C2; Description P/N Capacitor SMD 50V -> Capacitor SMD 25V
- C13: renamed from C9; Description P/N (none) -> Capacitor SMD 25V
- C14: renamed from C10; Description P/N (none) -> Capacitor SMD 25V
- C15: renamed from C11; Description P/N (none) -> Capacitor SMD 25V
- C16: renamed from C3; Description P/N Capacitor SMD 50V -> Capacitor SMD 25V
- C17: renamed from C4; Description P/N Capacitor SMD 50V -> Capacitor SMD 25V
- C18: renamed from C96; Description P/N (none) -> Capacitor SMD 25V
- C19: renamed from C97; Description P/N (none) -> Capacitor SMD 25V
- C2: renamed from C6; Description P/N (none) -> Capacitor SMD 25V
- C20: renamed from C104; Description P/N (none) -> Capacitor SMD 25V
- C21: renamed from C12; Description P/N Capacitor SMD 50V -> Capacitor SMD 25V
- C22: renamed from C13; Description P/N Capacitor SMD 50V -> Capacitor SMD 25V
- C23: renamed from C93; Description P/N (none) -> Capacitor SMD 25V
- C24: renamed from C92; Description P/N (none) -> Capacitor SMD 25V
- C25: renamed from C89; Description P/N (none) -> Capacitor SMD 25V
- C26: renamed from C88; Description P/N (none) -> Capacitor SMD 25V
- C27: renamed from C94; Description P/N (none) -> Capacitor SMD 25V
- C28: renamed from C95; Description P/N (none) -> Capacitor SMD 25V
- C29: renamed from C90; Description P/N (none) -> Capacitor SMD 25V
- C3: renamed from C7; Description P/N (none) -> Capacitor SMD 25V
- C30: renamed from C91; Description P/N (none) -> Capacitor SMD 25V
- C31: renamed from C99; Description P/N (none) -> Capacitor SMD 25V
- C32: renamed from C100; Description P/N (none) -> Capacitor SMD 25V
- C33: renamed from C18; Description P/N (none) -> Capacitor SMD 25V
- C34: renamed from C19; Description P/N (none) -> Capacitor SMD 25V
- C35: renamed from C20; Description P/N (none) -> Capacitor SMD 25V
- C36: renamed from C98; Description P/N (none) -> Capacitor SMD 25V
- C37: renamed from C21; Description P/N (none) -> Capacitor SMD 100V
- C38: renamed from C22; Description P/N (none) -> Capacitor electrolytic low ESR; Product Name (none) -> EEUFR2A101
- C39: renamed from C23; Description P/N (none) -> Capacitor SMD 100V
- C4: renamed from C8; Description P/N (none) -> Capacitor SMD 25V
- C40: renamed from C24; Description P/N (none) -> Capacitor SMD 50V
- C41: renamed from C25; Description P/N (none) -> Capacitor SMD 50V
- C42: renamed from C26; Description P/N (none) -> Capacitor electrolytic low ESR; Product Name (none) -> EEUFM1V221L
- C43: renamed from C101; Description P/N (none) -> Capacitor SMD 25V
- C44: renamed from C33; Description P/N (none) -> Capacitor SMD 25V
- C45: renamed from C34; Description P/N (none) -> Capacitor SMD 25V
- C46: renamed from C35; Description P/N (none) -> Capacitor SMD 25V
- C47: renamed from C36; Description P/N (none) -> Capacitor SMD 25V
- C48: renamed from C37; Description P/N (none) -> Capacitor SMD 25V
- C49: renamed from C38; Description P/N (none) -> Capacitor SMD 25V
- C5: renamed from C14; Description P/N (none) -> Capacitor SMD 25V
- C50: renamed from C39; Description P/N (none) -> Capacitor SMD 25V
- C51: renamed from C27; Description P/N (none) -> Capacitor SMD 50V
- C52: renamed from C28; Description P/N (none) -> Capacitor SMD 50V
- C53: renamed from C29; Description P/N (none) -> Capacitor SMD 50V
- C54: renamed from C30; Description P/N (none) -> Capacitor SMD 25V
- C55: renamed from C31; Description P/N (none) -> Capacitor SMD 25V
- C56: renamed from C32; Description P/N (none) -> Capacitor SMD 25V
- C6: renamed from C15; Description P/N (none) -> Capacitor SMD 25V
- C7: renamed from C16; Description P/N (none) -> Capacitor SMD 25V
- C8: renamed from C17; Description P/N (none) -> Capacitor SMD 25V
- D1: renamed from D2; value TD301MCANFD -> (none); Description P/N (none) -> CAN transiever; Product Name (none) -> TD301MCANFD
- D11: renamed from D8; value D_Schottky_Small -> (none); Description P/N (none) -> Diode; Product Name (none) -> US1B
- D12: renamed from D47; value D_Small -> (none); Description P/N (none) -> Diode; Product Name (none) -> GS3MB
- D13: renamed from D46; value D_TVS_Small -> (none); Description P/N (none) -> TVS; Product Name (none) -> SMBJ51A
- D14: renamed from D12; value D_TVS_Small -> (none); Description P/N (none) -> TVS; Product Name (none) -> SMCJ58A
- D15: renamed from D13; value D_Schottky_Small -> (none); Description P/N (none) -> Diode; Product Name (none) -> US1B
- D16: renamed from D14; value D_Schottky_Small -> (none); Description P/N (none) -> Diode; Product Name (none) -> US1B
- D17: renamed from D6; value K7809T -> (none); Description P/N (none) -> DC/DC; Product Name (none) -> K7809T
- D18: renamed from D7; value URB2415LD-20WR3 -> (none); Description P/N (none) -> DC/DC; Product Name (none) -> URB2415LD-20WR3
- D4: renamed from D26; value TD301MCANFD -> (none); Description P/N (none) -> CAN transiever; Product Name (none) -> TD301MCANFD
- J2: value Power_IN -> (none); Description P/N (none) -> Connector; Product Name (none) -> DS1073-01-2x2-MVT6
- L1: Description P/N (none) -> Inductor SMD; Product Name (none) -> ACM2520-301-2P-T002
- L2: renamed from L14; Description P/N (none) -> Inductor SMD; Product Name (none) -> ACM2520-301-2P-T002
- L3: renamed from L2; Description P/N (none) -> Inductor SMD; Product Name (none) -> ETQP4M100KVC
- L4: renamed from L3; Description P/N (none) -> Inductor SMD; Product Name (none) -> ETQP4M100KVC
- Q1, Q2, Q3, Q4: value WMM043N10HGD -> (none); Description P/N (none) -> MOSFET; Product Name (none) -> WMM043N10HGD
- R1: renamed from R5; Description P/N (none) -> Resistor SMD 1%
- R10: renamed from R8; Description P/N Resistor SMD -> Resistor SMD 1%
- R11: renamed from R80; Description P/N (none) -> Resistor SMD 1%
- R12: renamed from R79; Description P/N (none) -> Resistor SMD 1%
- R13: renamed from R64; Description P/N (none) -> Resistor SMD 1%
- R14: renamed from R52; Description P/N (none) -> Resistor SMD 1%
- R15: renamed from R81; Description P/N (none) -> Resistor SMD 1%
- R16: renamed from R82; Description P/N (none) -> Resistor SMD 1%
- R17: renamed from R84; Description P/N (none) -> Resistor SMD 1%
- R18: renamed from R83; Description P/N (none) -> Resistor SMD 1%
- R19: renamed from R85; Description P/N (none) -> Resistor SMD 1%
- R2: renamed from R6; Description P/N (none) -> Resistor SMD 1%
- R20: renamed from R87; Description P/N (none) -> Resistor SMD 1%
- R21: renamed from R78; Description P/N (none) -> Resistor SMD 1%; Product Name (none) -> ERJP08F10R0V
- R22: renamed from R88; Description P/N (none) -> Resistor SMD 1%
- R23: renamed from R9; Description P/N (none) -> Resistor SMD 1%
- R24: renamed from R10; Description P/N (none) -> Resistor SMD 1%
- R25: renamed from R90; Description P/N (none) -> Resistor SMD 1%
- R26: renamed from R15; Description P/N (none) -> Resistor SMD 1%
- R27: renamed from R16; Description P/N (none) -> Resistor SMD 1%
- R28: renamed from R89; Description P/N (none) -> Resistor SMD 1%
- R29: renamed from R91; Description P/N (none) -> Resistor SMD 1%
- R3: renamed from R1; Description P/N Resistor SMD -> Resistor SMD 1%
- R30: renamed from R17; Description P/N (none) -> Resistor SMD 1%
- R31: renamed from R18; Description P/N (none) -> Resistor SMD 1%
- R32: renamed from R19; Description P/N (none) -> Resistor SMD 1%
- R33: renamed from R20; Description P/N (none) -> Resistor SMD 1%
- R34: renamed from R21; Description P/N (none) -> Resistor SMD 1%
- R35: renamed from R22; Description P/N (none) -> Resistor SMD 1%
- R36: renamed from R23; Description P/N (none) -> Resistor SMD 1%
- R37: renamed from R24; Description P/N (none) -> Resistor SMD 1%
- R38: renamed from R25; Description P/N (none) -> Resistor SMD 1%
- R39: renamed from R26; Description P/N (none) -> Resistor SMD 1%
- R4: renamed from R2; Description P/N Resistor SMD -> Resistor SMD 1%
- R40: renamed from R27; Description P/N (none) -> Resistor SMD 1%
- R41: renamed from R11; Description P/N (none) -> Resistor SMD 1%
- R42: renamed from R12; Description P/N (none) -> Resistor SMD 1%
- R43: renamed from R13; Description P/N (none) -> Resistor SMD 1%
- R44: renamed from R14; Description P/N (none) -> Resistor SMD 1%
- R45: renamed from R29; Description P/N (none) -> Resistor SMD 1%
- R46: renamed from R30; Description P/N (none) -> Resistor SMD 1%
- R5: renamed from R3; Description P/N Resistor SMD -> Resistor SMD 1%
- R6: renamed from R4; Description P/N Resistor SMD -> Resistor SMD 1%
- R7: renamed from R86; Description P/N (none) -> Resistor SMD 1%
- R8: renamed from R98; Description P/N (none) -> Resistor SMD 1%
- R9: renamed from R7; Description P/N Resistor SMD -> Resistor SMD 1%
- U1: Description P/N (none) -> FRAM
- U4: renamed from U17; value TLV3501AIDBV -> (none); Description P/N (none) -> Comparator; Product Name (none) -> TLV3501AIDBV
- U5: renamed from U19; value TLV3501AIDBV -> (none); Description P/N (none) -> Comparator; Product Name (none) -> TLV3501AIDBV
- U6: renamed from U20; value TLV3501AIDBV -> (none); Description P/N (none) -> Comparator; Product Name (none) -> TLV3501AIDBV
- U7: renamed from U6; value LM5176PWP -> (none); Description P/N (none) -> DC/DC; Product Name (none) -> LM5176PWP
- U8: renamed from U4; value AMS1117-5.0 -> (none); Description P/N (none) -> Linear regulator; Product Name (none) -> AMS1117-5.0
- U9: renamed from U5; value AMS1117-3.3 -> (none); Description P/N (none) -> Linear regulator; Product Name (none) -> AMS1117-3.3
- renumbered D42 to D10, D9 to D19, D3 to D2, D10 to D20, D11 to D21, D15 to D22, D16 to D23, D1 to D3, D45 to D5, D4 to D6, D5 to D7, D40 to D8, D41 to D9
Connections:
- net +3.3V: now also C10.1, FB1.2; no longer C23.1, C24.1, C27.1, C28.1, C31.1, C32.1, D10.2 (K), D8.2 (K), D9.2 (K), R13.1, R17.1, R25.1, U3.13 (VDDA), U4.4 (V+), U5.4 (V+), U6.4 (V+)
- net BkIN_1: now also U3.33 (PB12); no longer U3.22 (PA6)
- net BkIN_8: now also U3.22 (PA6); no longer U3.33 (PB12)
- net GND: now also C10.2, C9.2
- new net +3.3VA: C23.1, C24.1, C27.1, C28.1, C31.1, C32.1, C9.1, D10.2 (K), D8.2 (K), D9.2 (K), FB1.1, R13.1, R17.1, R25.1, U3.13 (VDDA), U4.4 (V+), U5.4 (V+), U6.4 (V+)

Commit message: VER1.0: раскидал компоненты на плате
Parts:
- added H1, H2, H3, H4: MountingHole, MountingHole:MountingHole_4.3mm_M4, symbol Mechanical:MountingHole
- added J10, J11, J12, J13: (no value), Connector_Molex:Molex_Mini-Fit_Jr_5569-04A2_2x02_P4.20mm_Horizontal, symbol Connector_Generic:Conn_02x02_Top_Bottom
- C38: value 100u -> 68u; Product Name EEUFR2A101 -> EEUFC2A680
- C52, C53: footprint Capacitor_SMD:C_1210_3225Metric_Pad1.33x2.70mm_HandSolder -> Capacitor_SMD:C_1206_3216Metric_Pad1.33x1.80mm_HandSolder
- J2: footprint Connector_Molex:Molex_Mini-Fit_Jr_5566-04A_2x02_P4.20mm_Vertical -> Connector_Molex:Molex_Mini-Fit_Jr_5569-04A2_2x02_P4.20mm_Horizontal
Connections:
- net CANH_1: now also J10.3 (Pin_3), J11.3 (Pin_3)
- net CANH_2: now also J12.3 (Pin_3), J13.3 (Pin_3)
- net CANL_1: now also J10.4 (Pin_4), J11.4 (Pin_4)
- net CANL_2: now also J12.4 (Pin_4), J13.4 (Pin_4)
- net GND_CAN1: now also J10.1 (Pin_1), J10.2 (Pin_2), J11.1 (Pin_1), J11.2 (Pin_2)
- net GND_CAN2: now also J12.1 (Pin_1), J12.2 (Pin_2), J13.1 (Pin_1), J13.2 (Pin_2)
- net GND_IN: now also J2.1 (Pin_1); no longer J2.4 (Pin_4)
- net OverVoltage: now also U3.61 (PB8)
- net VIN: now also J2.4 (Pin_4); no longer J2.1 (Pin_1)
Other:
- moved on the sheet: J2

Commit message: VER1.0: отредактировал BOM
Parts:
- J10, J11, J12, J13, J2: Product Name DS1073-01-2x2-MVT6 -> DS1073-01-2x2MR2T6
Changed lines of the file:
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@@
 			)
 		)
-		(property "Product Name" "DS1073-01-2x2-MVT6"
+		(property "Product Name" "DS1073-01-2x2MR2T6"
 			(at 430.53 116.84 0)
 			(hide yes)
@@
 			)
 		)
-		(property "Product Name" "DS1073-01-2x2-MVT6"
+		(property "Product Name" "DS1073-01-2x2MR2T6"
 			(at 31.75 328.93 0)
 			(hide yes)
@@
 			)
 		)
-		(property "Product Name" "DS1073-01-2x2-MVT6"
+		(property "Product Name" "DS1073-01-2x2MR2T6"
 			(at 430.53 133.35 0)
 			(hide yes)
@@
 			)
 		)
-		(property "Product Name" "DS1073-01-2x2-MVT6"
+		(property "Product Name" "DS1073-01-2x2MR2T6"
 			(at 430.53 71.12 0)
 			(hide yes)
@@
 			)
 		)
-		(property "Product Name" "DS1073-01-2x2-MVT6"
+		(property "Product Name" "DS1073-01-2x2MR2T6"
 			(at 430.53 54.61 0)
 			(hide yes)
