File: PSFB_MCU.kicad_sch (KiCad schematic)
At the start: 154 parts, among them Y1 16M

Commit message: VER1.0: начал разводить плату
Connections:
- net GND1 is gone; now on net GND: D18.6 (0V), R42.2
Changed lines of the file:
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@@
 	)
 	(junction
+		(at 238.76 392.43)
+		(diameter 0)
+		(color 0 0 0 0)
+	)
+	(junction
 		(at 334.01 278.13)
 		(diameter 0)
@@
 	)
 	(junction
-		(at 238.76 392.43)
-		(diameter 0)
-		(color 0 0 0 0)
-	)
-	(junction
 		(at 393.7 344.17)
 		(diameter 0)
@@
 	)
 	(symbol
+		(lib_id "power:GND")
+		(at 238.76 392.43 0)
+		(unit 1)
+		(body_style 1)
+		(exclude_from_sim no)
+		(in_bom yes)
+		(on_board yes)
+		(in_pos_files yes)
+		(dnp no)
+		(property "Reference" "#PWR0133"
+			(at 238.76 398.78 0)
+			(hide yes)
+			(show_name no)
+			(do_not_autoplace no)
+			(effects
+				(font
+					(size 1.27 1.27)
+				)
+			)
+		)
+		(property "Value" "GND"
+			(at 238.76 396.24 0)
+			(show_name no)
+			(do_not_autoplace no)
+			(effects
+				(font
+					(size 1.27 1.27)
+				)
+			)
+		)
+		(property "Footprint" ""
+			(at 238.76 392.43 0)
+			(hide yes)
+			(show_name no)
+			(do_not_autoplace no)
+			(effects
+				(font
+					(size 1.27 1.27)
+				)
+			)
+		)
+		(property "Datasheet" ""
+			(at 238.76 392.43 0)
+			(hide yes)
+			(show_name no)
+			(do_not_autoplace no)
+			(effects
+				(font
+					(size 1.27 1.27)
+				)
+			)
+		)
+		(property "Description" "Power symbol creates a global label with name \"GND\" , ground"
+			(at 238.76 392.43 0)
+			(hide yes)
+			(show_name no)
+			(do_not_autoplace no)
+			(effects
+				(font
+					(size 1.27 1.27)
+				)
+			)
+		)
+		(pin "1"
+		)
+		(instances
+			(project "PSFB_MCU"
+				(path "/1f44d793-713f-4781-bd7e-20142de81965"
+					(reference "#PWR0133")
+					(unit 1)
+				)
+			)
+		)
+	)
+	(symbol
 		(lib_id "Device:C_Small")
 		(at 199.39 49.53 0)
@@
 					(unit 1)
 				)
-			)
-		)
-	)
-	(symbol
-		(lib_id "power:GND1")
-		(at 238.76 392.43 0)
-		(unit 1)
-		(body_style 1)
-		(exclude_from_sim no)
-		(in_bom yes)
-		(on_board yes)
-		(in_pos_files yes)
-		(dnp no)
-		(property "Reference" "#PWR0115"
-			(at 238.76 398.78 0)
-			(hide yes)
-			(show_name no)
-			(do_not_autoplace no)
-			(effects
-				(font
-					(size 1.27 1.27)
-				)
-			)
-		)
-		(property "Value" "GND1"
-			(at 238.76 396.748 0)
-			(show_name no)
-			(do_not_autoplace no)
-			(effects
-				(font
-					(size 1.27 1.27)
-				)
-			)
-		)
-		(property "Footprint" ""
-			(at 238.76 392.43 0)
-			(hide yes)
-			(show_name no)
-			(do_not_autoplace no)
-			(effects
-				(font
-					(size 1.27 1.27)
-				)
-			)
-		)
-		(property "Datasheet" ""
-			(at 238.76 392.43 0)
-			(hide yes)
-			(show_name no)
-			(do_not_autoplace no)
-			(effects
-				(font
-					(size 1.27 1.27)
-				)
-			)
-		)
-		(property "Description" "Power symbol creates a global label with name \"GND1\" , ground"
-			(at 238.76 392.43 0)
-			(hide yes)
-			(show_name no)
-			(do_not_autoplace no)
-			(effects
-				(font
-					(size 1.27 1.27)
-				)
-			)
-		)
-		(pin "1"
-		)
-		(instances
-			(project "PSFB_MCU"
-				(path "/1f44d793-713f-4781-bd7e-20142de81965"
-					(reference "#PWR0115")
-					(unit 1)
-				)

Commit message: VER1.0: развел плату, сделал гербера и BOM
Parts:
- removed C10: 10u, Capacitor_SMD:C_0805_2012Metric_Pad1.18x1.45mm_HandSolder, symbol Device:C_Small
- added FB4, FB5, FB6: (no value), Inductor_SMD:L_0805_2012Metric_Pad1.05x1.20mm_HandSolder, symbol Device:FerriteBead_Small
Connections:
- net +3.3V: now also D10.2 (K), D8.2 (K), D9.2 (K), R13.1, R17.1, R25.1, FB4.1, FB5.1, FB6.1
- net +3.3VA: no longer C23.1, C24.1, C27.1, C28.1, C31.1, C32.1, D10.2 (K), D8.2 (K), D9.2 (K), R13.1, R17.1, R25.1, U4.4 (V+), U5.4 (V+), U6.4 (V+)
- net ERROR_Channel_1: now also U3.4 (PC15)
- net ERROR_Channel_2: now also U3.56 (PB4)
- net RST_Channel_1: now also U3.62 (PB9)
- net RST_Channel_2: now also U3.54 (PD2)
- new net: C31.1, C32.1, FB6.2, U6.4 (V+)
- new net: C23.1, C24.1, FB4.2, U4.4 (V+)
- new net: C27.1, C28.1, FB5.2, U5.4 (V+)
- no-connect marks 5 -> 16
Other:
- moved on the sheet: D6, D7, R10, R9

Commit message: VER1.0: обновил гербера и BOM
Parts:
- added C107: 10p, Capacitor_SMD:C_0805_2012Metric_Pad1.18x1.45mm_HandSolder, symbol Device:C_Small
- added D48: (no value), Package_TO_SOT_SMD:SOT-23, symbol Device:D_Dual_Series_AKC_Parallel
- added J14: (no value), Connector_PinHeader_2.54mm:PinHeader_2x02_P2.54mm_Vertical, symbol Connector_Generic:Conn_02x02_Odd_Even
- added R47: 100, Resistor_SMD:R_0805_2012Metric_Pad1.20x1.40mm_HandSolder, symbol Device:R_Small
- U2: Product Name USBLC6-2P6 -> USBLC6-2SC6
Connections:
- net +3.3V: now also D48.2 (K)
- net GND: now also C107.2, D48.1 (A), J14.3 (Pin_3), J14.4 (Pin_4)
- net TMR2_CH2_SYNC: now reaches U3.55 (PB3)
- net TMR2_CH2_SYNC: now also C107.1, D48.3 (common), R47.1
- new net: J14.1 (Pin_1), J14.2 (Pin_2), R47.2
- no-connect marks 16 -> 15
