File: LV_measure.kicad_sch (KiCad schematic)
At the start: 39 parts

Commit message: VER1.0: добавил разделение питания VDD и VDDA
Parts:
- C100: renamed from C85; Description P/N Capacitor SMD 50V -> Capacitor SMD 25V
- C101: renamed from C77; Description P/N Capacitor SMD 50V -> Capacitor SMD 25V
- C102: renamed from C79; Description P/N Capacitor SMD 50V -> Capacitor SMD 25V
- C103: renamed from C81; Description P/N Capacitor SMD 50V -> Capacitor SMD 25V
- C104: renamed from C82; Description P/N Capacitor SMD 50V -> Capacitor SMD 25V
- C90: renamed from C73; Description P/N Capacitor SMD 50V -> Capacitor SMD 25V
- C92: renamed from C76; Description P/N Capacitor SMD 50V -> Capacitor SMD 25V
- C93: renamed from C78; Description P/N Polarized capacitor -> Capacitor tantalum SMD 6.3V; Product Name 293D107X96R3B2TE3 -> 6TPE100MWB
- C94: renamed from C80; Description P/N Capacitor SMD 50V -> Capacitor SMD 25V
- C95: renamed from C83; Description P/N Capacitor SMD 50V -> Capacitor SMD 25V
- C96: renamed from C84; Description P/N Capacitor SMD 50V -> Capacitor SMD 25V
- C97: renamed from C86; Description P/N Capacitor SMD 50V -> Capacitor SMD 25V
- C98: renamed from C75; Description P/N Capacitor SMD 50V -> Capacitor SMD 25V
- C99: renamed from C87; Description P/N Capacitor SMD 50V -> Capacitor SMD 25V
- R80: renamed from R74; Description P/N Resistor SMD -> Resistor SMD 1%
- R81: renamed from R66; Description P/N Resistor SMD -> Resistor SMD 0.1%
- R82: renamed from R67; Description P/N Resistor SMD -> Resistor SMD 0.1%
- R83: renamed from R68; Description P/N Resistor SMD -> Resistor SMD 0.1%
- R84: renamed from R75; Description P/N Resistor SMD -> Resistor SMD 1%
- R85: renamed from R69; Description P/N Resistor SMD -> Resistor SMD 0.1%
- R86: renamed from R65; Description P/N Resistor SMD -> Resistor SMD 1%
- R87: renamed from R71; Description P/N Resistor SMD -> Resistor SMD 1%
- R88: renamed from R72; Description P/N Resistor SMD -> Resistor SMD 1%
- R89: renamed from R70; Description P/N Resistor SMD -> Resistor SMD 0.1%
- R90: renamed from R77; Description P/N Resistor SMD -> Resistor SMD 1%
- R91: renamed from R73; Description P/N Resistor SMD -> Resistor SMD 1%
- R92: renamed from R76; Description P/N Resistor SMD -> Resistor SMD 1%
- U21: renamed from U16; Product Name OPA333xxDBV -> OPA333AIDBVR
- renumbered C74 to C91, D37 to D39, D34 to D40, D35 to D41, D38 to D42, D36 to D43, D33 to D44, D32 to D45, J6 to J7, L13 to L14, U32 to U20
Connections:
- net +3.3V renamed +3.3VA

Commit message: VER1.0: раскидал компоненты на плате
Parts:
- C93: footprint Capacitor_Tantalum_SMD:CP_EIA-3528-21_Kemet-B_Pad1.50x2.35mm_HandSolder -> Capacitor_Tantalum_SMD:CP_EIA-3528-21_Kemet-B_HandSolder
- J7: footprint Connector_My:Mini-Fit_01x02_Vertical -> Connector_Molex:Molex_Mini-Fit_Jr_5569-02A2_2x01_P4.20mm_Horizontal
Connections:
- net +3.3VP renamed +3V3

Commit message: VER1.0: отредактировал BOM
Parts:
- J7: Product Name DS1073-01-2x1-MVT6 -> DS1073-01-2x1MR2T6
Changed lines of the file:
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@@
 			)
 		)
-		(property "Product Name" "DS1073-01-2x1-MVT6"
+		(property "Product Name" "DS1073-01-2x1MR2T6"
 			(at 99.06 110.49 0)
 			(hide yes)
