File: LV_measure.kicad_sch (KiCad schematic)
At the start: 39 parts

Commit message: VER1.0: развел плату, сделал гербера и BOM
Parts:
- added FB7, FB8: (no value), Inductor_SMD:L_0805_2012Metric_Pad1.05x1.20mm_HandSolder, symbol Device:FerriteBead_Small
Connections:
- net +3.3VA: no longer names the net of C103.2, C104.1, D43.8 (VDD2)
- net +3.3VA: now also FB7.2; no longer C97.1, D42.2 (K), U21.5 (V+)
- new net: C97.1, FB8.2, U21.5 (V+)
- new net +3.3V: D42.2 (K), FB7.1, FB8.1
Other:
- moved on the sheet: C103, C104
