File: HV_measure.kicad_sch (KiCad schematic)
At the start: 42 parts

Commit message: VER1.0: развел плату, сделал гербера и BOM
Parts:
- added FB2, FB3: (no value), Inductor_SMD:L_0805_2012Metric_Pad1.05x1.20mm_HandSolder, symbol Device:FerriteBead_Small
Connections:
- net +3.3VA: no longer names the net of C88.2, C89.1, D38.8 (VDD2)
- net +3.3VA: now also FB2.2; no longer C82.1, D35.2 (K), U19.5 (V+)
- new net: C82.1, FB3.2, U19.5 (V+)
- new net +3.3V: D35.2 (K), FB2.1, FB3.1
Other:
- moved on the sheet: C88, C89
