File: PSFB_MCU.kicad_pcb (KiCad board)
At the start: 4 copper layers, 179 x 99 mm, 277 parts, among them Y1 16M

Commit message: VER1.0: начал разводить плату
Parts:
- moved D23 35.8 mm to (66.0, 103.5)
- moved R46 35.8 mm to (66.0, 103.5)
- moved C35 2.67 mm to (97.0, 73.5), turned to 90 degrees
- moved C45 2.67 mm to (99.5, 73.5)
- moved C34 2.36 mm to (86.5, 81.0), turned to -90 degrees
- moved R35 0.96 mm to (86.5, 77.0), turned to -90 degrees
Connections:
- D18 pad 6: GND1 -> GND
- R42 pad 2: GND1 -> GND
Routing:
- net /LDRV1: track 0.00 -> 52.2 mm, vias 0 -> 2
- net /SW1: track 0.00 -> 51.6 mm, vias 0 -> 45
- net /HDRV1: track 0.00 -> 47.3 mm, vias 0 -> 2
- net GND_IN: track 0.00 -> 44.0 mm, vias 0 -> 38
- net +24V: track 0.00 -> 27.5 mm, vias 0 -> 10
- net /SW2: track 0.00 -> 26.4 mm, vias 0 -> 46
- net /LDRV2: track 0.00 -> 23.6 mm, vias 0 -> 2
- net /HDRV2: track 0.00 -> 22.0 mm, vias 0 -> 2
- net VCC: track 0.00 -> 17.0 mm, vias 0 -> 1
- net GND: track 0.00 -> 9.57 mm, vias 0 -> 2
- net Net-(U7-SS): track 0.00 -> 7.46 mm, vias 0 -> 1
- net Net-(U7-COMP): track 0.00 -> 7.15 mm
- net Net-(U7-CS): track 0.00 -> 6.46 mm
- net Net-(U7-CSG): track 0.00 -> 5.94 mm
- net Net-(D16-K): track 0.00 -> 5.88 mm
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- added copper zone on F.Cu, net +15V
- added copper zone on B.Cu, net +24V
- added copper zone on F.Cu, net +24V
- added copper zone on B.Cu, net /SW1
- added copper zone on F.Cu, net /SW1
- added copper zone on In2.Cu, net /SW1
- added copper zone on B.Cu, net /SW2
- added copper zone on F.Cu, net /SW2
- added copper zone on In2.Cu, net /SW2
- added copper zone on In1.Cu, net GND
- added copper zone on B.Cu, net GND_IN
- added copper zone on F.Cu, net GND_IN
- added copper zone on In1.Cu, net GND_IN
- added copper zone on In2.Cu, net GND_IN
- added copper zone on B.Cu, net Net-(D12-K)
- added copper zone on F.Cu, net Net-(D12-K)
- added copper zone on In2.Cu, net Net-(D12-K)
- added copper zone on B.Cu, net Net-(D14-A2)
- added copper zone on F.Cu, net Net-(D14-A2)
- added copper zone on In2.Cu, net Net-(D14-A2)
- added copper zone on B.Cu, net Net-(Q3-S)
- added copper zone on F.Cu, net Net-(Q3-S)
- added copper zone on In2.Cu, net Net-(Q3-S)
- added copper zone on F.Cu, net VIN

Commit message: VER1.0: развел плату, сделал гербера и BOM
Parts:
- removed C10: 10u, Capacitor_SMD:C_0805_2012Metric_Pad1.18x1.45mm_HandSolder
- added FB2: ~, Inductor_SMD:L_0805_2012Metric_Pad1.05x1.20mm_HandSolder, B.Cu at (138.5, 95.0)
- added FB3: ~, Inductor_SMD:L_0805_2012Metric_Pad1.05x1.20mm_HandSolder, B.Cu at (144.5, 86.0)
- added FB4: ~, Inductor_SMD:L_0805_2012Metric_Pad1.05x1.20mm_HandSolder, F.Cu at (114.0, 89.0)
- added FB5: ~, Inductor_SMD:L_0805_2012Metric_Pad1.05x1.20mm_HandSolder, F.Cu at (178.0, 107.5)
- added FB6: ~, Inductor_SMD:L_0805_2012Metric_Pad1.05x1.20mm_HandSolder, F.Cu at (193.0, 107.5)
- added FB7: ~, Inductor_SMD:L_0805_2012Metric_Pad1.05x1.20mm_HandSolder, B.Cu at (118.0, 95.0)
- added FB8: ~, Inductor_SMD:L_0805_2012Metric_Pad1.05x1.20mm_HandSolder, B.Cu at (124.0, 86.0)
- C9, FB1: moved to B.Cu
- D34, D41, D8: moved to F.Cu
- moved C9 48.8 mm to (148.2, 79.0), turned to 180 degrees
- moved FB1 46.1 mm to (151.0, 80.0), turned to -90 degrees
- moved D13 23.3 mm to (92.5, 92.5), turned to 90 degrees
- moved R21 17.0 mm to (92.5, 87.5), turned to 0 degrees
- moved C35 13.3 mm to (86.0, 81.0), turned to -90 degrees
- moved D8 11.7 mm to (128.0, 90.5)
- moved D19 11.5 mm to (204.0, 94.5), turned to 180 degrees
- moved R41 11.5 mm to (204.0, 94.5), turned to 180 degrees
- moved C54 10.0 mm to (204.0, 84.0)
- moved D34 6.58 mm to (145.0, 108.0), turned to 180 degrees
- moved R4 5.70 mm to (144.0, 78.5)
- moved D3 4.25 mm to (176.5, 75.8)
- moved D6 4.25 mm to (151.0, 63.8)
- moved D7 4.25 mm to (148.5, 63.8)
- moved J1 4.25 mm to (180.5, 68.2)
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Connections:
- C103 pad 2: +3.3VA -> Net-(D43-VDD2)
- C104 pad 1: +3.3VA -> Net-(D43-VDD2)
- C23 pad 1: +3.3VA -> Net-(U4-V+)
- C24 pad 1: +3.3VA -> Net-(U4-V+)
- C27 pad 1: +3.3VA -> Net-(U5-V+)
- C28 pad 1: +3.3VA -> Net-(U5-V+)
- C31 pad 1: +3.3VA -> Net-(U6-V+)
- C32 pad 1: +3.3VA -> Net-(U6-V+)
- C82 pad 1: +3.3VA -> Net-(U19-V+)
- C88 pad 2: +3.3VA -> Net-(D38-VDD2)
- C89 pad 1: +3.3VA -> Net-(D38-VDD2)
- C97 pad 1: +3.3VA -> Net-(U21-V+)
- D10 pad 2: +3.3VA -> +3.3V
- D35 pad 2: +3.3VA -> +3.3V
- D38 pad 8: +3.3VA -> Net-(D38-VDD2)
- D42 pad 2: +3.3VA -> +3.3V
- D43 pad 8: +3.3VA -> Net-(D43-VDD2)
- D46 pad 2: +3.3VA -> +3.3V
- D47 pad 2: +3.3VA -> +3.3V
- D8 pad 2: +3.3VA -> +3.3V
- D9 pad 2: +3.3VA -> +3.3V
- R13 pad 1: +3.3VA -> +3.3V
- R17 pad 1: +3.3VA -> +3.3V
- R25 pad 1: +3.3VA -> +3.3V
- U19 pad 5: +3.3VA -> Net-(U19-V+)
- U21 pad 5: +3.3VA -> Net-(U21-V+)
- U3 pad 4: unconnected-(U3-PC15-Pad4) -> /ERROR_Channel_1
- U3 pad 54: unconnected-(U3-PD2-Pad54) -> /RST_Channel_2
- U3 pad 56: unconnected-(U3-PB4-Pad56) -> /ERROR_Channel_2
- U3 pad 62: unconnected-(U3-PB9-Pad62) -> /RST_Channel_1
- U4 pad 4: +3.3VA -> Net-(U4-V+)
- U5 pad 4: +3.3VA -> Net-(U5-V+)
- U6 pad 4: +3.3VA -> Net-(U6-V+)
Routing:
- net GND: track 9.57 -> 170.0 mm, vias 2 -> 91
- net +3.3V: track 0.00 -> 124.1 mm, vias 0 -> 69
- net /TMR1_CH2: track 0.00 -> 118.5 mm, vias 0 -> 2
- net /TMR1_CH1N: track 0.00 -> 118.4 mm, vias 0 -> 2
- net /TMR1_CH2N: track 0.00 -> 113.6 mm, vias 0 -> 4
- net /TMR1_CH1: track 0.00 -> 110.7 mm, vias 0 -> 2
- net /RST_Channel_1: track 0.00 -> 96.0 mm, vias 0 -> 2
- net /SHDN_OverCurrent_2: track 0.00 -> 89.2 mm, vias 0 -> 3
- net /OverVoltage: track 0.00 -> 86.0 mm, vias 0 -> 3
- net /ERROR_Channel_1: track 0.00 -> 82.2 mm, vias 0 -> 2
- net /CAN2_RXD_MCU: track 0.00 -> 81.4 mm, vias 0 -> 1
- net /SHDN_OverCurrent_1: track 0.00 -> 72.9 mm, vias 0 -> 3
- net /CAN2_TXD_MCU: track 0.00 -> 72.5 mm, vias 0 -> 1
- net /Current_measure_2: track 0.00 -> 70.9 mm, vias 0 -> 3
- net +3V3: track 0.00 -> 68.9 mm, vias 0 -> 23
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- added copper zone on In2.Cu, net +15V
- added copper zone on F.Cu, net +3.3V
- added copper zone on In2.Cu, net +3.3V
- added copper zone on B.Cu, net +3.3VP
- added copper zone on F.Cu, net +3.3VP
- added copper zone on B.Cu, net +3V3
- added copper zone on F.Cu, net +3V3
- added copper zone on B.Cu, net +5V
- added copper zone on F.Cu, net +5V
- added copper zone on F.Cu, net +9V
- added copper zone on B.Cu, net GND
- added copper zone on F.Cu, net GND
- added copper zone on B.Cu, net GNDPWR
- added copper zone on In1.Cu, net GNDPWR
- added copper zone on In1.Cu, net GND_CAN1
- added copper zone on In1.Cu, net GND_CAN2
- added copper zone on B.Cu, net GND_OUT
- added copper zone on In2.Cu, net GND_OUT
Other:
- outline, holes or cut-outs redrawn
- board text added: "+"
- board text added: "+15V"
- board text added: "+24V"
- board text added: "+3.3V"
- board text added: "+5V"
- board text added: "+VDC"
- board text added: "-"
- board text added: "12V"
- board text added: "CAN1"
- board text added: "CAN2"
- board text added: "Current1"
- board text added: "Current2"
- board text added: "G"
- board text added: "GND"
- board text added: "GNDPWR"
- board text added: "H"
- board text added: "L"
- board text added: "OUT"
- board text added: "SWCLK"
- board text added: "SWDIO"
- board text added: "USER LEDs"
- board text added: "VIN"
