File: PSFB_MCU.kicad_pcb (KiCad board)
At the start: 4 copper layers, 179 x 99 mm, 283 parts, among them Y1 16M

Commit message: VER1.0: обновил гербера и BOM
Parts:
- added C107: 10p, Capacitor_SMD:C_0805_2012Metric_Pad1.18x1.45mm_HandSolder, F.Cu at (197.2, 62.0)
- added D48: ~, Package_TO_SOT_SMD:SOT-23, F.Cu at (193.6, 60.7)
- added J14: ~, Connector_PinHeader_2.54mm:PinHeader_2x02_P2.54mm_Vertical, F.Cu at (201.5, 59.7)
- added R47: 100, Resistor_SMD:R_0805_2012Metric_Pad1.20x1.40mm_HandSolder, F.Cu at (197.2, 59.8)
- moved R3 1.25 mm to (156.2, 65.0)
Connections:
- U3 pad 55: unconnected-(U3-PB3-Pad55) -> /TMR2_CH2_SYNC
Routing:
- net /TMR2_CH2_SYNC: track 0.00 -> 46.2 mm, vias 0 -> 2
- net Net-(J14-Pin_1): track 0.00 -> 5.78 mm
- net GND: track 170.0 -> 174.5 mm, vias 91 -> 92
- net BOOT0: track 4.08 -> 5.39 mm
- net +3.3V: track 124.1 -> 125.2 mm, vias 69 -> 70
Other:
- board text added: "TMR"
- board text added: "TMR SYNC"
